File: tankbot/circuit/CIRCUIT.sch (EAGLE design)
At the start: 19 parts, among them X1 KUSBVX

Commit message: PCBfinal
Connections:
- removed net N$6: C1.+, IC2.IN
- net VIN: now also C1.+, IC2.IN
Changed lines of the file:
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@@
 <setting verticaltext="up"/>
 </settings>
-<grid distance="25" unitdist="mil" unit="mil" style="lines" multiple="1" display="no" altdistance="0.01" altunitdist="inch" altunit="inch"/>
+<grid distance="0.1" unitdist="inch" unit="inch" style="lines" multiple="1" display="no" altdistance="0.01" altunitdist="inch" altunit="inch"/>
 <layers>
 <layer number="1" name="Top" color="4" fill="1" visible="no" active="no"/>
@@
 <classes>
 <class number="0" name="default" width="0.381" drill="0.2032">
-<clearance class="0" value="0.889"/>
+<clearance class="0" value="1.27"/>
 </class>
 <class number="1" name="RasPins" width="0" drill="8">
-<clearance class="1" value="0.889"/>
+<clearance class="1" value="1.27"/>
 </class>
 <class number="2" name="TivaPins" width="0.381" drill="0.2032">
-<clearance class="2" value="0.889"/>
-</class>
-<class number="3" name="VInbat" width="0.762" drill="0.2032">
-<clearance class="3" value="0.889"/>
-</class>
-<class number="4" name="5v3A" width="0.635" drill="0.2032">
-<clearance class="4" value="0.889"/>
+<clearance class="2" value="1.27"/>
+</class>
+<class number="3" name="VInbat" width="1.27" drill="0.4064">
+<clearance class="3" value="1.27"/>
+</class>
+<class number="4" name="5v3A" width="1.27" drill="0.508">
+<clearance class="4" value="1.27"/>
 </class>
 <class number="5" name="outsVoltaje" width="0.635" drill="0.2032">
-<clearance class="5" value="0.889"/>
+<clearance class="5" value="1.27"/>
 </class>
 </classes>
@@
 </segment>
 <segment>
-<label x="58.42" y="-22.86" size="1.778" layer="95" rot="MR0" xref="yes"/>
-</segment>
-<segment>
 <pinref part="D1" gate="1" pin="C"/>
 <wire x1="129.54" y1="35.56" x2="137.16" y2="35.56" width="0.1524" layer="91"/>
@@
 <junction x="154.94" y="-35.56"/>
 <label x="157.48" y="-35.56" size="0.8128" layer="95" rot="MR180" xref="yes"/>
+</segment>
+<segment>
+<pinref part="C1" gate="G$1" pin="+"/>
+<pinref part="IC2" gate="A" pin="IN"/>
+<wire x1="63.5" y1="-27.94" x2="63.5" y2="-22.86" width="0.1524" layer="91"/>
+<wire x1="63.5" y1="-22.86" x2="71.12" y2="-22.86" width="0.1524" layer="91"/>
+<label x="60.96" y="-22.86" size="1.778" layer="95" rot="MR0" xref="yes"/>
 </segment>
 </net>
@@
 </segment>
 </net>
-<net name="N$6" class="0">
-<segment>
-<pinref part="C1" gate="G$1" pin="+"/>
-<pinref part="IC2" gate="A" pin="IN"/>
-<wire x1="63.5" y1="-27.94" x2="63.5" y2="-22.86" width="0.1524" layer="91"/>
-<wire x1="63.5" y1="-22.86" x2="71.12" y2="-22.86" width="0.1524" layer="91"/>
-<wire x1="58.42" y1="-22.86" x2="63.5" y2="-22.86" width="0.1524" layer="91"/>
-<junction x="63.5" y="-22.86"/>
-</segment>
-</net>
