File: tankbot/circuit/CIRCUIT.brd (EAGLE design)
At the start: 78.7 x 140.6 mm, 19 parts, among them X1 KUSBVX

Commit message: PCBfinal
Parts:
- moved D1 1.91 mm to (-17.8, -74.3)
Connections:
- removed net N$6: C1.+, IC2.3
- net VIN: now also C1.+, IC2.3
Routing:
- net VIN: track 88.1 -> 139.7 mm, vias 0 -> 2
- net N$6: track 33.2 -> 0.00 mm
- net 3V31A: track 170.6 -> 183.3 mm
- net GND@1: track 329.0 -> 333.4 mm
- net PL4: track 89.8 -> 91.8 mm
- net PL5: track 72.6 -> 74.4 mm
- net PK4: track 29.8 -> 31.5 mm
- net PK5: track 26.2 -> 27.1 mm
- net N$2: track 9.94 -> 9.15 mm
- net N$1: track 20.4 -> 19.7 mm

Commit message: FINAL BOARD
Connections:
- removed net PL4: U$1.P16, U$2.P1
- removed net PL5: U$1.P15, U$2.P7
- new net PF2: U$1.P19, U$2.P1
- new net PF3: U$1.P18, U$2.P7
Routing:
- net PF2: track 0.00 -> 98.9 mm
- net PL4: track 91.8 -> 0.00 mm
- net PF3: track 0.00 -> 81.5 mm, vias 0 -> 2
- net PL5: track 74.4 -> 0.00 mm, vias 2 -> 0
- net GND@1: track 333.4 -> 330.4 mm
Changed lines of the file:
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@@
 </element>
 <element name="U$1" library="TivaConnector" package="TIVAPINESPCB" value="TIVAEKTM4C" x="-16.51" y="39.37" smashed="yes" rot="MR0">
+<attribute name="NAME" x="-13.208" y="53.043665625" size="1.27" layer="26" rot="MR0"/>
+<attribute name="NAME" x="-56.388" y="-10.456334375" size="1.27" layer="26" rot="MR0"/>
+<attribute name="NAME" x="-13.208" y="-10.456334375" size="1.27" layer="26" rot="MR0"/>
 <attribute name="NAME" x="-56.388" y="53.043665625" size="1.27" layer="26" rot="MR0"/>
-<attribute name="NAME" x="-13.208" y="-10.456334375" size="1.27" layer="26" rot="MR0"/>
-<attribute name="NAME" x="-56.388" y="-10.456334375" size="1.27" layer="26" rot="MR0"/>
-<attribute name="NAME" x="-13.208" y="53.043665625" size="1.27" layer="26" rot="MR0"/>
+<attribute name="VALUE" x="-13.208" y="-39.073665625" size="1.27" layer="28" rot="MR0"/>
 <attribute name="VALUE" x="-13.208" y="24.426334375" size="1.27" layer="28" rot="MR0"/>
+<attribute name="VALUE" x="-56.388" y="24.426334375" size="1.27" layer="28" rot="MR0"/>
 <attribute name="VALUE" x="-56.388" y="-39.073665625" size="1.27" layer="28" rot="MR0"/>
-<attribute name="VALUE" x="-13.208" y="-39.073665625" size="1.27" layer="28" rot="MR0"/>
-<attribute name="VALUE" x="-56.388" y="24.426334375" size="1.27" layer="28" rot="MR0"/>
 </element>
 <element name="X1" library="con-kycon" library_urn="urn:adsk.eagle:library:157" package="KUSBVX" package3d_urn="urn:adsk.eagle:package:7682/1" value="KUSBVX" x="-50.8" y="-76.2" smashed="yes" rot="R180">
@@
 <wire x1="-13.97" y1="-66.04" x2="-28.575" y2="-66.04" width="1.27" layer="16"/>
 <wire x1="-28.575" y1="-66.04" x2="-50.8" y2="-43.815" width="1.27" layer="16"/>
-<wire x1="-50.8" y1="-43.815" x2="-50.8" y2="-15.24" width="1.27" layer="16"/>
-<wire x1="-50.8" y1="-15.24" x2="-45.847" y2="-10.287" width="1.27" layer="16"/>
-<wire x1="-45.847" y1="-10.287" x2="-45.847" y2="-10.16" width="1.27" layer="16"/>
+<wire x1="-50.8" y1="-43.815" x2="-50.8" y2="-14.859" width="1.27" layer="16"/>
+<wire x1="-50.8" y1="-14.859" x2="-46.101" y2="-10.16" width="1.27" layer="16"/>
 <contactref element="C1" pad="+"/>
 <contactref element="IC2" pad="3"/>
@@
 <wire x1="-13.97" y1="-66.04" x2="-13.97" y2="-60.96" width="1.27" layer="16"/>
 <via x="-13.97" y="-60.96" extent="1-16" drill="0.762" diameter="2.286"/>
-<wire x1="-45.847" y1="-10.16" x2="-45.72" y2="-10.16" width="0" layer="19" extent="16-16"/>
+<wire x1="-46.101" y1="-10.16" x2="-45.72" y2="-10.16" width="1.27" layer="16"/>
 </signal>
 <signal name="GND@1" class="5">
@@
 <wire x1="7.62" y1="38.1" x2="7.62" y2="30.48" width="0.762" layer="16"/>
 <wire x1="-40.3606" y1="-7.65305625" x2="-42.315184375" y2="-5.698471875" width="0.762" layer="16"/>
-<wire x1="-58.42" y1="-15.24" x2="-58.1406" y2="-15.5194" width="0.762" layer="16"/>
-<wire x1="-55.5244" y1="-15.5194" x2="-58.1406" y2="-15.5194" width="0.762" layer="16"/>
 <wire x1="-40.64" y1="-10.16" x2="-40.3606" y2="-9.8806" width="0.762" layer="16"/>
 <wire x1="-40.3606" y1="-7.65305625" x2="-40.3606" y2="-9.8806" width="0.762" layer="16"/>
-<wire x1="-42.315184375" y1="-5.698471875" x2="-46.219128125" y2="-5.698471875" width="0.762" layer="16"/>
+<wire x1="-42.315184375" y1="-5.698471875" x2="-45.965128125" y2="-5.698471875" width="0.762" layer="16"/>
 <wire x1="8.89" y1="-20.32" x2="8.89" y2="-22.86" width="0.762" layer="16"/>
 <wire x1="8.89" y1="-20.32" x2="8.89" y2="-17.78" width="0.762" layer="16"/>
@@
 <wire x1="-9.5758" y1="-69.85" x2="-9.5758" y2="-47.5742" width="1.27" layer="16"/>
 <wire x1="-9.5758" y1="-47.5742" x2="-13.97" y2="-43.18" width="1.27" layer="16"/>
-<wire x1="-58.42" y1="-15.24" x2="-55.76065625" y2="-15.24" width="0.762" layer="16"/>
 <wire x1="-56.06545625" y1="-15.24" x2="-55.5244" y2="-15.78105625" width="0.762" layer="16"/>
-<wire x1="-55.76065625" y1="-15.24" x2="-46.219128125" y2="-5.698471875" width="0.762" layer="16"/>
-<wire x1="-55.5244" y1="-15.5194" x2="-56.06545625" y2="-15.24" width="0" layer="19" extent="16-16"/>
+<wire x1="-58.42" y1="-15.24" x2="-56.06545625" y2="-15.24" width="0.762" layer="16"/>
+<wire x1="-55.50665625" y1="-15.24" x2="-56.06545625" y2="-15.24" width="0.762" layer="16"/>
+<wire x1="-45.965128125" y1="-5.698471875" x2="-55.50665625" y2="-15.24" width="0.762" layer="16"/>
 </signal>
 <signal name="5V3A" class="4">
@@
 <contactref element="U$1" pad="P33"/>
 </signal>
-<signal name="PL4" class="2">
-<contactref element="U$1" pad="P16"/>
-<contactref element="U$2" pad="P1"/>
-<wire x1="-37.465" y1="-13.335" x2="-26.67" y2="-13.335" width="0.762" layer="16"/>
-<wire x1="-26.67" y1="-13.335" x2="-24.765" y2="-11.43" width="0.762" layer="16"/>
-<wire x1="-24.765" y1="-11.43" x2="-24.765" y2="19.685" width="0.762" layer="16"/>
-<wire x1="-24.765" y1="19.685" x2="-31.115" y2="26.035" width="0.762" layer="16"/>
-<wire x1="-31.115" y1="26.035" x2="-31.115" y2="31.75" width="0.762" layer="16"/>
-<wire x1="-31.115" y1="31.75" x2="-22.225" y2="40.64" width="0.762" layer="16"/>
-<wire x1="-22.225" y1="40.64" x2="-17.78" y2="40.64" width="0.762" layer="16"/>
-<wire x1="-37.465" y1="-13.335" x2="-45.72" y2="-21.59" width="0.762" layer="16"/>
-<wire x1="-45.72" y1="-21.59" x2="-45.72" y2="-25.4" width="0.762" layer="16"/>
-</signal>
-<signal name="PL5" class="2">
-<contactref element="U$1" pad="P15"/>
-<contactref element="U$2" pad="P7"/>
-<wire x1="-17.78" y1="38.1" x2="-20.32" y2="38.1" width="0.762" layer="16"/>
-<wire x1="-20.32" y1="38.1" x2="-24.765" y2="33.655" width="0.762" layer="16"/>
-<wire x1="-24.765" y1="33.655" x2="-24.13" y2="33.02" width="0.762" layer="16"/>
-<wire x1="-28.82134375" y1="-22.225" x2="-30.48" y2="-23.88365625" width="0.762" layer="16"/>
-<wire x1="-30.48" y1="-25.4" x2="-30.48" y2="-23.88365625" width="0.762" layer="16"/>
-<wire x1="-24.13" y1="-22.86" x2="-24.765" y2="-22.225" width="0.762" layer="16"/>
-<wire x1="-24.765" y1="-22.225" x2="-28.82134375" y2="-22.225" width="0.762" layer="16"/>
-<via x="-24.13" y="-22.86" extent="1-16" drill="0.762" diameter="2.286"/>
-<wire x1="-24.13" y1="-22.86" x2="-24.13" y2="33.02" width="0.762" layer="1"/>
-<via x="-24.13" y="33.02" extent="1-16" drill="0.762" diameter="2.286"/>
-</signal>
 <signal name="N$10">
 <contactref element="U$2" pad="P13"/>
@@
 </polygon>
 </signal>
+<signal name="PF2">
+<contactref element="U$1" pad="P19"/>
+<contactref element="U$2" pad="P1"/>
+<wire x1="-37.465" y1="-13.335" x2="-26.67" y2="-13.335" width="0.762" layer="16"/>
+<wire x1="-26.67" y1="-13.335" x2="-24.765" y2="-11.43" width="0.762" layer="16"/>
+<wire x1="-24.765" y1="-11.43" x2="-24.765" y2="19.685" width="0.762" layer="16"/>
+<wire x1="-24.765" y1="19.685" x2="-31.115" y2="26.035" width="0.762" layer="16"/>
+<wire x1="-31.115" y1="26.035" x2="-31.115" y2="31.75" width="0.762" layer="16"/>
+<wire x1="-31.115" y1="31.75" x2="-24.384" y2="38.481" width="0.762" layer="16"/>
+<wire x1="-37.465" y1="-13.335" x2="-45.72" y2="-21.59" width="0.762" layer="16"/>
+<wire x1="-45.72" y1="-21.59" x2="-45.72" y2="-25.4" width="0.762" layer="16"/>
+<wire x1="-24.384" y1="38.481" x2="-24.384" y2="45.212" width="0.762" layer="16"/>
+<wire x1="-24.384" y1="45.212" x2="-21.336" y2="48.26" width="0.762" layer="16"/>
+<wire x1="-21.336" y1="48.26" x2="-17.78" y2="48.26" width="0.762" layer="16"/>
+</signal>
+<signal name="PF3">
+<contactref element="U$1" pad="P18"/>
+<contactref element="U$2" pad="P7"/>
+<wire x1="-24.765" y1="33.655" x2="-21.717" y2="36.703" width="0.762" layer="16"/>
+<wire x1="-24.765" y1="33.655" x2="-24.13" y2="33.02" width="0.762" layer="16"/>
+<wire x1="-28.82134375" y1="-22.225" x2="-30.48" y2="-23.88365625" width="0.762" layer="16"/>
+<wire x1="-30.48" y1="-25.4" x2="-30.48" y2="-23.88365625" width="0.762" layer="16"/>
+<wire x1="-24.13" y1="-22.86" x2="-24.765" y2="-22.225" width="0.762" layer="16"/>
+<wire x1="-24.765" y1="-22.225" x2="-28.82134375" y2="-22.225" width="0.762" layer="16"/>
+<via x="-24.13" y="-22.86" extent="1-16" drill="0.762" diameter="2.286"/>
+<wire x1="-24.13" y1="-22.86" x2="-24.13" y2="33.02" width="0.762" layer="1"/>
+<via x="-24.13" y="33.02" extent="1-16" drill="0.762" diameter="2.286"/>
+<wire x1="-21.717" y1="43.34045625" x2="-19.40095625" y2="45.6565" width="0.762" layer="16"/>
+<wire x1="-21.717" y1="43.34045625" x2="-21.717" y2="36.703" width="0.762" layer="16"/>
+<wire x1="-19.40095625" y1="45.6565" x2="-17.8435" y2="45.6565" width="0.762" layer="16"/>
+<wire x1="-17.8435" y1="45.6565" x2="-17.78" y2="45.72" width="0.381" layer="16"/>
+</signal>
 </signals>
